Commit message: diff robot urdf finished

File: urdf/diff_robot.urdf (robot description, URDF)
Before this commit: robot robot_name, 2 links, 1 joints
Links:
- removed link /* child_link */
- removed link /* parent_link */
- added link base_link, mass 0.0; collision box size=0 0 0; visual box size=0.8 0.7 0.1
- added link wheel_rear_left_link, mass 0.0; collision cylinder length=0.1 radius=0.15; visual cylinder length=0.1 radius=0.15
- added link wheel_rear_right_link, mass 0.0; collision cylinder length=0.1 radius=0.15; visual cylinder length=0.1 radius=0.15
Joints:
- removed joint /* joint_name */
- added joint wheel_rear_left_joint: type continuous, parent base_link, child wheel_rear_left_link, origin xyz=0.250 -0.4 0 rpy=1.57 0 0, axis 0 0 0
- added joint wheel_rear_right_joint: type continuous, parent base_link, child wheel_rear_right_link, origin xyz=0.250 0.4 0 rpy=1.57 0 0, axis 0 0 0
