Commit message: added diff robot to rviz

File: mobile_robot/urdf/diff_robot.urdf (robot description, URDF)
Before this commit: robot diff_robot, 3 links, 2 joints
Links:
- added link base_footprint
Joints:
- added joint base_joint: type fixed, parent base_footprint, child base_link, origin xyz=0 0 0.135 rpy=0 0 0, axis 0 0 0
- joint wheel_rear_left_joint: axis 0 0 0 -> 0 0 1
- joint wheel_rear_right_joint: axis 0 0 0 -> 0 0 1
