Commit message: urdf file changed to xacro

File: mobile_robot/urdf/diff_robot.xacro (robot description, xacro)
@@ -1,4 +1,4 @@
 <?xml version="1.0"?>
-<robot name="diff_robot">
+<robot xmlns:xacro="http://ww.ros.org/wiki/xacro" name="diff_robot">
     <link name="base_footprint">
     </link>
@@ -29,6 +29,8 @@
         <axis xyz="0 0 0"/>
     </joint>
-    <!-- Rear Right Wheel -->
-    <link name="wheel_rear_right_link">
+    <!-- Right Wheel -->
+    <xacro:property name='side' value='right'/>
+    <xacro:property name='reflect' value='1'/>
+    <link name="wheel_${side}_link">
         <visual>
             <geometry>
@@ -50,12 +52,14 @@
         </inertial>
     </link>
-    <joint name="wheel_rear_right_joint" type="continuous">
+    <joint name="wheel_${side}_joint" type="continuous">
         <parent link="base_link"/>
-        <child link="wheel_rear_right_link"/>
-        <origin xyz="0.250 0.4 0" rpy="1.57 0 0"/>
+        <child link="wheel_${side}_link"/>
+        <origin xyz="0.250 ${reflect*0.4} 0" rpy="1.57 0 0"/>
         <axis xyz="0 0 1"/>
     </joint>
     <!-- Rear Left Wheel -->
-    <link name="wheel_rear_left_link">
+    <xacro:property name='side' value='left'/>
+    <xacro:property name='reflect' value='-1'/>
+    <link name="wheel_${side}_link">
         <visual>
             <geometry>
@@ -77,8 +81,8 @@
         </inertial>
     </link>
-    <joint name="wheel_rear_left_joint" type="continuous">
+    <joint name="wheel_${side}_joint" type="continuous">
         <parent link="base_link"/>
-        <child link="wheel_rear_left_link"/>
-        <origin xyz="0.250 -0.4 0" rpy="1.57 0 0"/>
+        <child link="wheel_${side}_link"/>
+        <origin xyz="0.250 ${reflect*0.4} 0" rpy="1.57 0 0"/>
         <axis xyz="0 0 1"/>
     </joint>

Commit message: added macro to the xacro

File: mobile_robot/urdf/diff_robot.xacro (robot description, xacro)
@@ -29,61 +29,35 @@
         <axis xyz="0 0 0"/>
     </joint>
-    <!-- Right Wheel -->
-    <xacro:property name='side' value='right'/>
-    <xacro:property name='reflect' value='1'/>
-    <link name="wheel_${side}_link">
-        <visual>
-            <geometry>
-                <cylinder radius="0.15" length="0.1"/>
-            </geometry>
-            <material name="Red">
-                <color rgba="1. 0. 0. 1"/>
-            </material>
-        </visual>
-        <collision>
-            <geometry>
-                <cylinder radius="0.15" length="0.1"/>
-            </geometry>
-        </collision>
-        <inertial>
-            <mass value="0.0"/>
-            <origin xyz="0.0 0.0 0.0" rpy="0.0 0.0 0.0"/>
-            <inertia ixx="0.0" ixy="0.0" ixz="0.0" iyy="0.0" iyz="0.0" izz="0.0"/>
-        </inertial>
-    </link>
-    <joint name="wheel_${side}_joint" type="continuous">
-        <parent link="base_link"/>
-        <child link="wheel_${side}_link"/>
-        <origin xyz="0.250 ${reflect*0.4} 0" rpy="1.57 0 0"/>
-        <axis xyz="0 0 1"/>
-    </joint>
-    <!-- Rear Left Wheel -->
-    <xacro:property name='side' value='left'/>
-    <xacro:property name='reflect' value='-1'/>
-    <link name="wheel_${side}_link">
-        <visual>
-            <geometry>
-                <cylinder radius="0.15" length="0.1"/>
-            </geometry>
-            <material name="Red">
-                <color rgba="1. 0. 0. 1"/>
-            </material>
-        </visual>
-        <collision>
-            <geometry>
-                <cylinder radius="0.15" length="0.1"/>
-            </geometry>
-        </collision>
-        <inertial>
-            <mass value="0.0"/>
-            <origin xyz="0.0 0.0 0.0" rpy="0.0 0.0 0.0"/>
-            <inertia ixx="0.0" ixy="0.0" ixz="0.0" iyy="0.0" iyz="0.0" izz="0.0"/>
-        </inertial>
-    </link>
-    <joint name="wheel_${side}_joint" type="continuous">
-        <parent link="base_link"/>
-        <child link="wheel_${side}_link"/>
-        <origin xyz="0.250 ${reflect*0.4} 0" rpy="1.57 0 0"/>
-        <axis xyz="0 0 1"/>
-    </joint>
+    <xacro:macro name='wheel' params='name x y'>
+        <link name="wheel_${name}_link">
+            <visual>
+                <geometry>
+                    <cylinder radius="0.15" length="0.1"/>
+                </geometry>
+                <material name="Red">
+                    <color rgba="1. 0. 0. 1"/>
+                </material>
+            </visual>
+            <collision>
+                <geometry>
+                    <cylinder radius="0.15" length="0.1"/>
+                </geometry>
+            </collision>
+            <inertial>
+                <mass value="0.0"/>
+                <origin xyz="0.0 0.0 0.0" rpy="0.0 0.0 0.0"/>
+                <inertia ixx="0.0" ixy="0.0" ixz="0.0" iyy="0.0" iyz="0.0" izz="0.0"/>
+            </inertial>
+        </link>
+        <joint name="wheel_${name}_joint" type="continuous">
+            <parent link="base_link"/>
+            <child link="wheel_${name}_link"/>
+            <origin xyz="${x} ${y} 0" rpy="1.57 0 0"/>
+            <axis xyz="0 0 1"/>
+        </joint>
+    </xacro:macro>
+    <!-- Right wheel-->
+    <xacro:wheel name="right" x="0.250" y="0.40"/>
+    <!-- Left Wheel -->
+    <xacro:wheel name="left" x="0.250" y="-0.40"/>
 </robot>

Commit message: changed frames in urdf to match mobro convention and some code cleaning

File: mobile_robot/urdf/diff_robot.xacro (robot description, xacro)
@@ -1,4 +1,5 @@
 <?xml version="1.0"?>
 <robot xmlns:xacro="http://ww.ros.org/wiki/xacro" name="diff_robot">
+    <xacro:property name="pi" value="3.14159265359"/>
     <link name="base_footprint">
     </link>
@@ -11,4 +12,5 @@
                 <color rgba="0.7 0.7 0.7 1.0"/>
             </material>
+            <origin xyz="0.250 0.0 0.0" rpy="0.0 0.0 0.0"/>
         </visual>
         <collision>
@@ -53,5 +55,5 @@
             <parent link="base_link"/>
             <child link="wheel_${name}_link"/>
-            <origin xyz="${x} ${y} 0" rpy="1.57 0 0"/>
+            <origin xyz="${x} ${y} 0" rpy="${-pi/2} 0 0"/>
             <axis xyz="0 0 1"/>
         </joint>

Commit message: removed pi property declaration

File: mobile_robot/urdf/diff_robot.xacro (robot description, xacro)
@@ -1,5 +1,4 @@
 <?xml version="1.0"?>
 <robot xmlns:xacro="http://ww.ros.org/wiki/xacro" name="diff_robot">
-    <xacro:property name="pi" value="3.14159265359"/>
     <link name="base_footprint">
     </link>

Commit message: made everything in xacro a variable

File: mobile_robot/urdf/diff_robot.xacro (robot description, xacro)
@@ -1,4 +1,7 @@
 <?xml version="1.0"?>
 <robot xmlns:xacro="http://ww.ros.org/wiki/xacro" name="diff_robot">
+    <xacro:property name="height_offset" value="0.135" />
+    <xacro:property name="wheel_radius" value="0.15" />
+    <xacro:property name="wheel_thickness" value="0.1" />
     <link name="base_footprint">
     </link>
@@ -27,12 +30,12 @@
         <parent link="base_footprint"/>
         <child link="base_link"/>
-        <origin xyz="0 0 0.135" rpy="0 0 0"/>
+        <origin xyz="0 0 ${height_offset}" rpy="0 0 0"/>
         <axis xyz="0 0 0"/>
     </joint>
-    <xacro:macro name='wheel' params='name x y'>
+    <xacro:macro name='wheel' params='name x_offset wheel_separation'>
         <link name="wheel_${name}_link">
             <visual>
                 <geometry>
-                    <cylinder radius="0.15" length="0.1"/>
+                    <cylinder radius="${wheel_radius}" length="${wheel_thickness}"/>
                 </geometry>
                 <material name="Red">
@@ -42,5 +45,5 @@
             <collision>
                 <geometry>
-                    <cylinder radius="0.15" length="0.1"/>
+                    <cylinder radius="${wheel_radius}" length="${wheel_thickness}"/>
                 </geometry>
             </collision>
@@ -54,11 +57,11 @@
             <parent link="base_link"/>
             <child link="wheel_${name}_link"/>
-            <origin xyz="${x} ${y} 0" rpy="${-pi/2} 0 0"/>
+            <origin xyz="${x_offset} ${wheel_separation/2} 0" rpy="${-pi/2} 0 0"/>
             <axis xyz="0 0 1"/>
         </joint>
     </xacro:macro>
     <!-- Right wheel-->
-    <xacro:wheel name="right" x="0" y="0.40"/>
+    <xacro:wheel name="right" x_offset="0" wheel_separation="0.80"/>
     <!-- Left Wheel -->
-    <xacro:wheel name="left" x="0" y="-0.40"/>
+    <xacro:wheel name="left" x_offset="0" wheel_separation="-0.80"/>
 </robot>

Commit message: added castor wheel

File: mobile_robot/urdf/diff_robot.xacro (robot description, xacro)
@@ -2,6 +2,10 @@
 <robot xmlns:xacro="http://ww.ros.org/wiki/xacro" name="diff_robot">
     <xacro:property name="height_offset" value="0.135" />
+    <xacro:property name="chassis_length" value="0.8" />
+    <xacro:property name="chassis_width" value="0.7" />
+    <xacro:property name="chassis_height" value="0.1" />
     <xacro:property name="wheel_radius" value="0.15" />
     <xacro:property name="wheel_thickness" value="0.1" />
+    <xacro:property name="castor_radius" value="0.05" />
     <link name="base_footprint">
     </link>
@@ -9,5 +13,5 @@
         <visual>
             <geometry>
-                <box size="0.8 0.7 0.1" />
+                <box size="${chassis_length} ${chassis_width} ${chassis_height}" />
             </geometry>
             <material name="LightGrey">
@@ -61,4 +65,30 @@
         </joint>
     </xacro:macro>
+    <link name="castor_link">
+        <visual>
+            <geometry>
+                <sphere radius="${castor_radius}"/>
+            </geometry>
+            <material name="LightGrey">
+                <color rgba="0.7 0.7 0.7 1.0"/>
+            </material>
+        </visual>
+        <collision>
+            <geometry>
+                <sphere radius="${castor_radius}"/>
+            </geometry>
+        </collision>
+        <inertial>
+            <mass value="0.0"/>
+            <origin xyz="0.0 0.0 0.0" rpy="0.0 0.0 0.0"/>
+            <inertia ixx="0.0" ixy="0.0" ixz="0.0" iyy="0.0" iyz="0.0" izz="0.0"/>
+        </inertial>
+    </link>
+    <joint name="castor_joint" type="fixed">
+        <parent link="base_link"/>
+        <child link="castor_link"/>
+        <origin xyz="0.55 0 ${-height_offset + castor_radius/2}" rpy="0 0 0"/>
+        <axis xyz="0 0 0"/>
+    </joint>
     <!-- Right wheel-->
     <xacro:wheel name="right" x_offset="0" wheel_separation="0.80"/>

Commit message: added castor_x_offset variable in xacro

File: mobile_robot/urdf/diff_robot.xacro (robot description, xacro)
@@ -8,4 +8,5 @@
     <xacro:property name="wheel_thickness" value="0.1" />
     <xacro:property name="castor_radius" value="0.05" />
+    <xacro:property name="castor_x_offset" value="0.55" />
     <link name="base_footprint">
     </link>
@@ -88,5 +89,5 @@
         <parent link="base_link"/>
         <child link="castor_link"/>
-        <origin xyz="0.55 0 ${-height_offset + castor_radius/2}" rpy="0 0 0"/>
+        <origin xyz="${castor_x_offset} 0 ${-height_offset + castor_radius/2}" rpy="0 0 0"/>
         <axis xyz="0 0 0"/>
     </joint>

Commit message: added calculation of inertias in xacro

File: mobile_robot/urdf/diff_robot.xacro (robot description, xacro)
@@ -1,12 +1,16 @@
 <?xml version="1.0"?>
 <robot xmlns:xacro="http://ww.ros.org/wiki/xacro" name="diff_robot">
+    <!-- Every value is in SI units -->
     <xacro:property name="height_offset" value="0.135" />
     <xacro:property name="chassis_length" value="0.8" />
     <xacro:property name="chassis_width" value="0.7" />
     <xacro:property name="chassis_height" value="0.1" />
+    <xacro:property name="chassis_mass" value="2" />
     <xacro:property name="wheel_radius" value="0.15" />
     <xacro:property name="wheel_thickness" value="0.1" />
+    <xacro:property name="wheel_mass" value="0.3" />
     <xacro:property name="castor_radius" value="0.05" />
     <xacro:property name="castor_x_offset" value="0.55" />
+    <xacro:property name="castor_mass" value="0.1" />
     <link name="base_footprint">
     </link>
@@ -29,5 +33,5 @@
             <mass value="0.0"/>
             <origin xyz="0.0 0.0 0.0" rpy="0.0 0.0 0.0"/>
-            <inertia ixx="0.0" ixy="0.0" ixz="0.0" iyy="0.0" iyz="0.0" izz="0.0"/>
+            <inertia ixx="${1/12*chassis_mass*(pow(chassis_height,2)+pow(chassis_length,2))}" ixy="0.0" ixz="0.0" iyy="${1/12*chassis_mass*(pow(chassis_width,2)+pow(chassis_height,2))}" iyz="0.0" izz="${1/12*chassis_mass*(pow(chassis_width,2)+pow(chassis_length,2))}"/>
         </inertial>
     </link>
@@ -54,7 +58,7 @@
             </collision>
             <inertial>
-                <mass value="0.0"/>
+                <mass value="0.2"/>
                 <origin xyz="0.0 0.0 0.0" rpy="0.0 0.0 0.0"/>
-                <inertia ixx="0.0" ixy="0.0" ixz="0.0" iyy="0.0" iyz="0.0" izz="0.0"/>
+                <inertia ixx="${1/12*wheel_mass*(3*pow(wheel_radius,2)+pow(wheel_thickness,2))}" ixy="0.0" ixz="0.0" iyy="${1/12*wheel_mass*(3*pow(wheel_radius,2)+pow(wheel_thickness,2))}" iyz="0.0" izz="${1/2*wheel_mass*pow(wheel_radius,2)}"/>
             </inertial>
         </link>
@@ -83,5 +87,5 @@
             <mass value="0.0"/>
             <origin xyz="0.0 0.0 0.0" rpy="0.0 0.0 0.0"/>
-            <inertia ixx="0.0" ixy="0.0" ixz="0.0" iyy="0.0" iyz="0.0" izz="0.0"/>
+            <inertia ixx="${2/5*castor_mass*pow(castor_radius,2)}" ixy="0.0" ixz="0.0" iyy="${2/5*castor_mass*pow(castor_radius,2)}" iyz="0.0" izz="${2/5*castor_mass*pow(castor_radius,2)}"/>
         </inertial>
     </link>

Commit message: fixed castor math bug

File: mobile_robot/urdf/diff_robot.xacro (robot description, xacro)
@@ -2,5 +2,5 @@
 <robot xmlns:xacro="http://ww.ros.org/wiki/xacro" name="diff_robot">
     <!-- Every value is in SI units -->
-    <xacro:property name="height_offset" value="0.135" />
+    <xacro:property name="height_offset" value="0.15" />
     <xacro:property name="chassis_length" value="0.8" />
     <xacro:property name="chassis_width" value="0.7" />
@@ -10,5 +10,5 @@
     <xacro:property name="wheel_thickness" value="0.1" />
     <xacro:property name="wheel_mass" value="0.3" />
-    <xacro:property name="castor_radius" value="0.05" />
+    <xacro:property name="castor_radius" value="0.045" />
     <xacro:property name="castor_x_offset" value="0.55" />
     <xacro:property name="castor_mass" value="0.1" />
@@ -31,5 +31,5 @@
         </collision>
         <inertial>
-            <mass value="0.0"/>
+            <mass value="${chassis_mass}"/>
             <origin xyz="0.0 0.0 0.0" rpy="0.0 0.0 0.0"/>
             <inertia ixx="${1/12*chassis_mass*(pow(chassis_height,2)+pow(chassis_length,2))}" ixy="0.0" ixz="0.0" iyy="${1/12*chassis_mass*(pow(chassis_width,2)+pow(chassis_height,2))}" iyz="0.0" izz="${1/12*chassis_mass*(pow(chassis_width,2)+pow(chassis_length,2))}"/>
@@ -58,5 +58,5 @@
             </collision>
             <inertial>
-                <mass value="0.2"/>
+                <mass value="${wheel_mass}"/>
                 <origin xyz="0.0 0.0 0.0" rpy="0.0 0.0 0.0"/>
                 <inertia ixx="${1/12*wheel_mass*(3*pow(wheel_radius,2)+pow(wheel_thickness,2))}" ixy="0.0" ixz="0.0" iyy="${1/12*wheel_mass*(3*pow(wheel_radius,2)+pow(wheel_thickness,2))}" iyz="0.0" izz="${1/2*wheel_mass*pow(wheel_radius,2)}"/>
@@ -85,5 +85,5 @@
         </collision>
         <inertial>
-            <mass value="0.0"/>
+            <mass value="${castor_mass}"/>
             <origin xyz="0.0 0.0 0.0" rpy="0.0 0.0 0.0"/>
             <inertia ixx="${2/5*castor_mass*pow(castor_radius,2)}" ixy="0.0" ixz="0.0" iyy="${2/5*castor_mass*pow(castor_radius,2)}" iyz="0.0" izz="${2/5*castor_mass*pow(castor_radius,2)}"/>
@@ -93,5 +93,5 @@
         <parent link="base_link"/>
         <child link="castor_link"/>
-        <origin xyz="${castor_x_offset} 0 ${-height_offset + castor_radius/2}" rpy="0 0 0"/>
+        <origin xyz="${castor_x_offset} 0 ${-height_offset + castor_radius}" rpy="0 0 0"/>
         <axis xyz="0 0 0"/>
     </joint>
