Commit message: added gazebo plugins in xacro

File: mobile_robot/description/diff_robot.xacro (robot description, xacro)
@@ -32,5 +32,5 @@
         <inertial>
             <mass value="${chassis_mass}"/>
-            <origin xyz="0.0 0.0 0.0" rpy="0.0 0.0 0.0"/>
+            <origin xyz="0.250 0.0 0.0" rpy="0.0 0.0 0.0"/>
             <inertia ixx="${1/12*chassis_mass*(pow(chassis_height,2)+pow(chassis_length,2))}" ixy="0.0" ixz="0.0" iyy="${1/12*chassis_mass*(pow(chassis_width,2)+pow(chassis_height,2))}" iyz="0.0" izz="${1/12*chassis_mass*(pow(chassis_width,2)+pow(chassis_length,2))}"/>
         </inertial>
@@ -100,3 +100,5 @@
     <!-- Left Wheel -->
     <xacro:wheel name="left" x_offset="0" wheel_separation="-0.80"/>
+    <!-- Include gazebo plugins -->
+    <xacro:include filename="gazebo.xacro" />
 </robot>
